File: ATTiny10DevBrd.brd (EAGLE design)
At the start: 46.7 x 45.7 mm, 15 parts, among them IC1 ATTINY10-MAHR

Commit message: Dev board and programmer adapter
Parts:
- removed 5VSEL: (no value), adafruit:1X03-CLEANBIG
- removed EXTPOWER: (no value), LL:1X04-SMD-LONG
- removed OUT: (no value), adafruit:2X04
- removed Q1: (no value), semicon-smd-ipc:SOT23
- added C4: 100uF, LL:PANASONIC_E
- added IC2: (no value), LL:SOT223
- added JP4: (no value), pinhead:2X02
- added JP5: (no value), pinhead:2X05
- added JP6: (no value), adafruit:1X01
- added L1: (no value), LL:L1812
- added R5: 0, LL:M0805
- added TP1, TP2, TP3, TP4, TP5, TP6, TP7, TP8, TP9: TPSQTP12R, testpad:TP12R
- C3: device adafruit:C0805 -> LL:C0805K
- R1: value 1K -> 100K
- R2: value BLANK -> (none); device adafruit:R0805 -> LL:M1206
- R3: value 1k -> (none); device adafruit:R0805 -> LL:M1206
- moved JP3 35.1 mm to (4.83, 10.7)
- moved JP1 17.1 mm to (19.8, 25.7), turned to 0 degrees
- moved C3 14.7 mm to (25.4, 21.8), turned to 180 degrees
- moved IC1 14.1 mm to (13.5, 20.1), turned to 270 degrees
- moved R1 12.2 mm to (6.86, 12.4)
- moved PRG 6.62 mm to (14.5, 13.7)
- moved C1 5.73 mm to (21.1, 20.6), turned to 90 degrees
- moved C2 5.39 mm to (18.8, 20.6), turned to 90 degrees
- moved R3 4.68 mm to (13.7, 24.6), turned to 270 degrees
- moved JP2 4.10 mm to (26.4, 10.4), turned to 0 degrees
- moved R2 2.27 mm to (10.4, 19.1)
Connections:
- removed net +12V: EXTPOWER.4, Q1.3
- removed net +5V: 5VSEL.2, C1.1, C2.1, C3.1, IC1.7, JP2.1, JP2.2, JP2.3
- removed net N$1: Q1.1, R2.2, R3.2
- removed net N$5: PRG.4, R1.2
- removed net VDD: 5VSEL.1, EXTPOWER.1
- new net VCC: C1.1, C2.1, IC1.7, JP6.1, L1.1, TP4.TP
- new net VIN: C4.+, IC2.3, JP4.1, JP4.2, TP6.TP
- net GND: now also C4.-, IC2.1, JP4.3, JP4.4, JP5.5, JP5.6, TP8.TP, TP9.TP; no longer EXTPOWER.2, EXTPOWER.3, OUT.7, OUT.8
- net PB2: now also JP5.7, JP5.8, R3.1, R3.2, TP5.TP; no longer OUT.5, OUT.6
- net PRGRST: now also IC1.6, R1.1, TP3.TP; no longer R2.1, R3.1
- net RST: now also JP5.10, JP5.9, R1.2; no longer IC1.6, Q1.2
- net TPICLK: now also JP5.3, JP5.4, R2.1, R2.2, TP2.TP; no longer OUT.3, OUT.4
- net TPIDATA: now also JP5.1, JP5.2, R5.1, R5.2, TP1.TP; no longer OUT.1, OUT.2, R1.1
- net V+: now also C3.1, IC2.2, JP2.1, JP2.2, JP2.3, L1.2, TP7.TP; no longer 5VSEL.3
Routing:
- net GND: track 9.12 -> 99.8 mm
- net N$1: track 63.7 -> 0.00 mm, vias 2 -> 0
- net +5V: track 62.8 -> 0.00 mm
- net PRGRST: track 13.8 -> 71.6 mm
- net TPIDATA: track 51.0 -> 19.5 mm, vias 2 -> 0
- net V+: track 9.28 -> 32.5 mm
- net RST: track 26.7 -> 8.43 mm, vias 2 -> 0
- net VIN: track 0.00 -> 15.6 mm
- net PB2: track 15.2 -> 30.7 mm, vias 2 -> 0
- net N$5: track 12.7 -> 0.00 mm, vias 2 -> 0
- net +12V: track 11.2 -> 0.00 mm
- net VCC: track 0.00 -> 10.9 mm
- net TPICLK: track 30.8 -> 21.5 mm, vias 2 -> 0
- net VDD: track 6.42 -> 0.00 mm
- added copper zone on layer 1, net N$1
- added copper zone on layer 1, net V+
- added copper zone on layer 1, net VCC
- added copper zone on layer 1, net VIN

Commit message: Tune traces
Parts:
- R3: value (none) -> 0
- R5: device LL:M0805 -> LL:R0805
Routing:
- net PRGRST: track 71.6 -> 72.7 mm
Changed lines of the file:
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@@
 <setting verticaltext="up"/>
 </settings>
-<grid distance="0.01" unitdist="inch" unit="inch" style="lines" multiple="1" display="yes" altdistance="0.025" altunitdist="inch" altunit="inch"/>
+<grid distance="0.005" unitdist="inch" unit="inch" style="lines" multiple="1" display="yes" altdistance="0.025" altunitdist="inch" altunit="inch"/>
 <layers>
 <layer number="1" name="Top" color="4" fill="1" visible="yes" active="yes"/>
@@
 </class>
 </classes>
-<designrules name="ll-etch *">
+<designrules name="ll-etch-lax">
 <description language="de">&lt;b&gt;EAGLE Design Rules&lt;/b&gt;
 &lt;p&gt;
@@
 <description language="en">&lt;b&gt;LL's Etch Rules&lt;/b&gt;
 &lt;p&gt;
-Toner transfer etch tuned DRU</description>
+Toner transfer etch tuned DRU
+(Most lax version designed to allow 8mil traces between 0805s and 0603s to even exist</description>
 <param name="layerSetup" value="(1*16)"/>
 <param name="mtCopper" value="0.0356mm 0.0356mm 0.0356mm 0.0356mm 0.0356mm 0.0356mm 0.0356mm 0.0356mm 0.0356mm 0.0356mm 0.0356mm 0.0356mm 0.0356mm 0.0356mm 0.0356mm 0.0356mm"/>
 <param name="mtIsolate" value="1.5011mm 0.1499mm 0.2007mm 0.1499mm 0.2007mm 0.1499mm 0.2007mm 0.1499mm 0.2007mm 0.1499mm 0.2007mm 0.1499mm 0.2007mm 0.1499mm 0.2007mm"/>
 <param name="mdWireWire" value="8mil"/>
-<param name="mdWirePad" value="12mil"/>
+<param name="mdWirePad" value="7mil"/>
 <param name="mdWireVia" value="12mil"/>
-<param name="mdPadPad" value="18mil"/>
+<param name="mdPadPad" value="12mil"/>
 <param name="mdPadVia" value="18mil"/>
 <param name="mdViaVia" value="20mil"/>
@@
 <param name="mdDrill" value="30mil"/>
 <param name="mdSmdStop" value="0mil"/>
-<param name="msWidth" value="10mil"/>
+<param name="msWidth" value="8mil"/>
 <param name="msDrill" value="21mil"/>
 <param name="msMicroVia" value="21mil"/>
@@
 <param name="rvMicroViaOuter" value="0.25"/>
 <param name="rvMicroViaInner" value="0.25"/>
-<param name="rlMinPadTop" value="15mil"/>
+<param name="rlMinPadTop" value="20mil"/>
 <param name="rlMaxPadTop" value="35mil"/>
 <param name="rlMinPadInner" value="20mil"/>
@@
 <param name="srMinRoundness" value="0mil"/>
 <param name="srMaxRoundness" value="0mil"/>
-<param name="slThermalIsolate" value="8mil"/>
+<param name="slThermalIsolate" value="10mil"/>
 <param name="slThermalsForVias" value="1"/>
 <param name="dpMaxLengthDifference" value="10mm"/>
@@
 <element name="JP5" library="pinhead" package="2X05" value="" x="12.954" y="6.604" rot="R180"/>
 <element name="R2" library="LL" package="M1206" value="" x="10.414" y="19.05" rot="R90"/>
-<element name="R5" library="LL" package="M0805" value="0" x="16.764" y="17.526" rot="R180"/>
-<element name="R3" library="LL" package="M1206" value="" x="13.716" y="24.638" rot="R270"/>
+<element name="R5" library="LL" package="R0805" value="0" x="16.764" y="17.526" rot="R180"/>
+<element name="R3" library="LL" package="M1206" value="0" x="13.716" y="24.638" rot="R270"/>
 <element name="JP6" library="adafruit" package="1X01" value="" x="22.86" y="19.304"/>
 <element name="TP1" library="testpad" package="TP12R" value="TPSQTP12R" x="20.828" y="6.604">
@@
 <wire x1="14.562" y1="20.816" x2="14.986" y2="21.336" width="0.3048" layer="1"/>
 <wire x1="14.986" y1="21.336" x2="15.229840625" y2="21.66111875" width="0.6096" layer="1"/>
-<contactref element="R3" pad="2"/>
-<contactref element="R3" pad="1"/>
-<wire x1="15.229840625" y1="21.66111875" x2="15.748" y2="22.352" width="0.6096" layer="1"/>
-<wire x1="13.716" y1="23.238" x2="15.229840625" y2="21.66111875" width="0.6096" layer="1"/>
-<wire x1="13.716" y1="26.038" x2="11.43" y2="25.654" width="0.4064" layer="1"/>
+<wire x1="15.229840625" y1="21.66111875" x2="15.3517625" y2="21.82368125" width="0.6096" layer="1"/>
+<wire x1="15.3517625" y1="21.82368125" x2="15.748" y2="22.352" width="0.6096" layer="1"/>
 <wire x1="11.43" y1="25.654" x2="7.62" y2="23.114" width="0.4064" layer="1"/>
 <wire x1="7.62" y1="23.114" x2="7.366" y2="18.288" width="0.4064" layer="1"/>
@@
 <wire x1="16.764" y1="22.098" x2="15.748" y2="22.098" width="0.4064" layer="1"/>
 <wire x1="15.748" y1="22.098" x2="15.748" y2="22.352" width="0.4064" layer="1"/>
+<contactref element="R3" pad="1"/>
+<contactref element="R3" pad="2"/>
+<wire x1="11.43" y1="25.654" x2="13.716" y2="26.038" width="0.6096" layer="1"/>
+<wire x1="13.716" y1="23.238" x2="15.3517625" y2="21.82368125" width="0.6096" layer="1"/>
 <wire x1="13.716" y1="26.038" x2="13.716" y2="23.238" width="0" layer="19" extent="1-1"/>
 </signal>
@@
 <wire x1="10.668" y1="21.082" x2="10.414" y2="20.45" width="0.4064" layer="1"/>
 <wire x1="14.478" y1="14.986" x2="13.208" y2="13.97" width="0.4064" layer="1"/>
-<wire x1="13.208" y1="13.97" x2="13.208" y2="10.922" width="0.4064" layer="1"/>
-<wire x1="13.208" y1="10.922" x2="15.494" y2="7.874" width="0.4064" layer="1"/>
+<wire x1="13.208" y1="13.97" x2="13.208" y2="11.43" width="0.4064" layer="1"/>
+<wire x1="13.208" y1="11.43" x2="15.494" y2="7.874" width="0.4064" layer="1"/>
 <wire x1="13.208" y1="13.97" x2="12.7" y2="13.716" width="0.4064" layer="1"/>
 <wire x1="12.7" y1="13.716" x2="10.668" y2="13.716" width="0.4064" layer="1"/>
@@
 <wire x1="18.034" y1="6.35" x2="18.034" y2="5.334" width="0.8128" layer="1"/>
 <wire x1="14.562" y1="19.316" x2="14.986" y2="19.05" width="0.254" layer="1"/>
-<wire x1="14.986" y1="19.05" x2="15.814" y2="17.526" width="0.4064" layer="1"/>
-<wire x1="17.714" y1="17.526" x2="17.526" y2="15.494" width="0.4064" layer="1"/>
+<wire x1="14.986" y1="19.05" x2="15.764" y2="17.526" width="0.4064" layer="1"/>
+<wire x1="17.764" y1="17.526" x2="17.526" y2="15.494" width="0.4064" layer="1"/>
 <wire x1="17.526" y1="15.494" x2="17.018" y2="14.986" width="0.4064" layer="1"/>
 <contactref element="TP1" pad="TP"/>
-<wire x1="20.828" y1="6.604" x2="18.034" y2="6.604" width="0.4064" layer="1"/>
+<wire x1="20.828" y1="6.604" x2="18.034" y2="6.604" width="0.6096" layer="1"/>
 <wire x1="18.034" y1="6.604" x2="18.034" y2="6.35" width="0.4064" layer="1"/>
-<wire x1="17.714" y1="17.526" x2="15.814" y2="17.526" width="0" layer="19" extent="1-1"/>
+<wire x1="17.764" y1="17.526" x2="15.764" y2="17.526" width="0" layer="19" extent="1-1"/>
 </signal>
 <signal name="GND">
@@
 <wire x1="6.858" y1="23.6728" x2="6.096" y2="18.0594" width="0.4064" layer="1"/>
 <wire x1="12.7" y1="28.2448" x2="6.858" y2="23.6728" width="0.4064" layer="1"/>
-<wire x1="26.6446" y1="28.2448" x2="12.7" y2="28.2448" width="0.4064" layer="1"/>
-<wire x1="25.4254" y1="23.368" x2="26.924" y2="23.876" width="0.4064" layer="1"/>
-<wire x1="26.924" y1="23.876" x2="26.6446" y2="28.2448" width="0.254" layer="1"/>
+<wire x1="26.7716" y1="28.2448" x2="12.7" y2="28.2448" width="0.4064" layer="1"/>
+<wire x1="25.4254" y1="23.368" x2="26.797" y2="24.003" width="0.4064" layer="1"/>
+<wire x1="26.797" y1="24.003" x2="26.7716" y2="28.2448" width="0.254" layer="1"/>
 <wire x1="25.4254" y1="19.2024" x2="25.4254" y2="23.368" width="0.254" layer="1"/>
 <wire x1="24.5872" y1="16.8402" x2="25.4254" y2="19.2024" width="0.6096" layer="1"/>
-<wire x1="24.5872" y1="13.8684" x2="24.5872" y2="16.8402" width="0.6096" layer="1"/>
-<wire x1="23.8252" y1="13.3604" x2="24.5872" y2="13.8684" width="0.4064" layer="1"/>
-<wire x1="21.5392" y1="13.3604" x2="23.8252" y2="13.3604" width="0.3048" layer="1"/>
+<wire x1="24.5872" y1="12.9794" x2="24.5872" y2="16.8402" width="0.6096" layer="1"/>
+<wire x1="23.6982" y1="12.8524" x2="24.5872" y2="12.9794" width="0.4064" layer="1"/>
+<wire x1="21.4122" y1="12.8524" x2="23.6982" y2="12.8524" width="0.6096" layer="1"/>
 <wire x1="20.7772" y1="16.9926" x2="20.5232" y2="14.478" width="0.6096" layer="1"/>
 <wire x1="20.5232" y1="14.478" x2="20.5232" y2="14.3764" width="0.3048" layer="1"/>
@@
 <wire x1="18.3388" y1="18.8976" x2="19.1262" y2="18.6436" width="0.254" layer="1"/>
 <wire x1="18.3388" y1="18.8976" x2="16.7259" y2="19.0627" width="0.254" layer="1"/>
-<wire x1="21.5392" y1="13.3604" x2="20.5232" y2="14.3764" width="0.4064" layer="1"/>
+<wire x1="21.4122" y1="12.8524" x2="20.5232" y2="14.3764" width="0.4064" layer="1"/>
 <contactref element="TP3" pad="TP"/>
 <wire x1="19.558" y1="15.748" x2="20.5232" y2="14.478" width="0.4064" layer="1"/>
@@
 <vertex x="25.654" y="13.208"/>
 <vertex x="27.432" y="27.178"/>
-<vertex x="28.956" y="27.178"/>
+<vertex x="28.702" y="27.178"/>
 <vertex x="29.21" y="9.398"/>
 <vertex x="21.336" y="9.398"/>
@@
 <polygon width="0.254" layer="1" spacing="0.6096" pour="hatch">
 <vertex x="29.464" y="27.178"/>
-<vertex x="29.464" y="20.066"/>
+<vertex x="29.718" y="20.066"/>
 <vertex x="30.226" y="19.304"/>
 <vertex x="43.434" y="19.05"/>
@@
 </signal>
 </signals>
+<errors>
+</errors>
 </board>
 </drawing>

Commit message: Tune up boards for printing
Parts:
- added U$1, U$2, U$3: (no value), holes:3,2
Other:
- board size 46.7 x 45.7 mm -> 46.7 x 38.3 mm
- board text added: "ATTiny10 Dev Brd v1.0 3/24/2013"
Changed lines of the file:
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@@
 <plain>
 <wire x1="0" y1="0" x2="46.66" y2="0" width="0" layer="20"/>
-<wire x1="46.66" y1="0" x2="46.66" y2="45.71" width="0" layer="20"/>
-<wire x1="46.66" y1="45.71" x2="0" y2="45.71" width="0" layer="20"/>
-<wire x1="0" y1="45.71" x2="0" y2="0" width="0" layer="20"/>
+<wire x1="46.66" y1="0" x2="46.533" y2="38.344" width="0" layer="20"/>
+<wire x1="46.533" y1="38.344" x2="0" y2="38.217" width="0" layer="20"/>
+<wire x1="0" y1="38.217" x2="0" y2="0" width="0" layer="20"/>
 <polygon width="0.254" layer="41">
 <vertex x="29.21" y="18.796"/>
@@
 <vertex x="37.338" y="18.796"/>
 </polygon>
+<text x="11.049" y="34.671" size="1.016" layer="1">ATTiny10 Dev Brd v1.0 3/24/2013</text>
 </plain>
 <attributes>
@@
 <attribute name="TP_SIGNAL_NAME" value="" x="21.336" y="30.734" size="1.778" layer="27" display="off"/>
 </element>
+<element name="U$1" library="holes" package="3,2" value="" x="5.08" y="33.02"/>
+<element name="U$2" library="holes" package="3,2" value="" x="40.64" y="33.147"/>
+<element name="U$3" library="holes" package="3,2" value="" x="40.64" y="5.08"/>
 </elements>
 <signals>
@@
 <polygon width="0.254" layer="1" spacing="0.6096" pour="hatch" isolate="0.4064" orphans="yes" rank="3">
 <vertex x="1.27" y="1.016"/>
-<vertex x="45.72" y="1.016"/>
-<vertex x="45.72" y="35.814"/>
-<vertex x="1.27" y="35.814"/>
+<vertex x="46.736" y="0.889"/>
+<vertex x="46.355" y="36.957"/>
+<vertex x="1.016" y="37.592"/>
 </polygon>
 <polygon width="0.254" layer="16" spacing="0.254" pour="hatch" isolate="0.254" orphans="yes">
 <vertex x="1.27" y="1.016"/>
-<vertex x="45.72" y="1.016"/>
-<vertex x="45.72" y="36.068"/>
-<vertex x="1.27" y="36.068"/>
+<vertex x="46.736" y="0.889"/>
+<vertex x="45.593" y="37.084"/>
+<vertex x="1.397" y="37.592"/>
 </polygon>
 <contactref element="IC2" pad="1"/>
@@
 <vertex x="43.434" y="19.05"/>
 <vertex x="42.418" y="22.098"/>
-<vertex x="37.338" y="27.178"/>
+<vertex x="33.147" y="27.051"/>
 </polygon>
 <contactref element="TP6" pad="TP"/>
@@
 </signal>
 </signals>
-<errors>
-</errors>
 </board>
 </drawing>
