File: ATTiny10ProgrammingAdapter.sch (EAGLE design)
At the start: 9 parts

Commit message: Fix rest to default to pulldown when not active
Parts:
- added R5: 50k, adafruit:R-US_R0805
- added R6: 2k, adafruit:R-US_R0805
Connections:
- new net N$4: Q1.C, R5.1
- net +12V: now also R5.2; no longer Q1.C
- net GND: now also R6.1
- net RST: now also R6.2
Changed lines of the file:
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@@
 <part name="VDD2" library="supply1" deviceset="VDD" device=""/>
 <part name="R4" library="LL" deviceset="R-US_" device="R1206" value="0"/>
+<part name="R5" library="adafruit" deviceset="R-US_" device="R0805" value="50k"/>
+<part name="GND3" library="supply1" deviceset="GND" device=""/>
+<part name="R6" library="adafruit" deviceset="R-US_" device="R0805" value="2k"/>
 </parts>
 <sheets>
@@
 <instance part="GND4" gate="1" x="111.76" y="12.7"/>
 <instance part="Q1" gate="G$1" x="48.26" y="68.58"/>
-<instance part="P+6" gate="1" x="50.8" y="81.28"/>
+<instance part="P+6" gate="1" x="50.8" y="93.98"/>
 <instance part="R2" gate="G$1" x="38.1" y="63.5"/>
 <instance part="R3" gate="G$1" x="38.1" y="71.12"/>
@@
 <instance part="VDD2" gate="G$1" x="83.82" y="83.82"/>
 <instance part="R4" gate="G$1" x="7.62" y="50.8"/>
+<instance part="R5" gate="G$1" x="50.8" y="83.82" rot="R90"/>
+<instance part="GND3" gate="1" x="50.8" y="43.18"/>
+<instance part="R6" gate="G$1" x="50.8" y="55.88" rot="R90"/>
 </instances>
 <busses>
@@
 <net name="RST" class="0">
 <segment>
-<pinref part="Q1" gate="G$1" pin="E"/>
-<wire x1="50.8" y1="63.5" x2="50.8" y2="60.96" width="0.1524" layer="91"/>
-<wire x1="50.8" y1="60.96" x2="53.34" y2="60.96" width="0.1524" layer="91"/>
-<label x="53.34" y="60.96" size="1.778" layer="95" xref="yes"/>
-</segment>
-<segment>
 <pinref part="PRG" gate="J" pin="RST"/>
 <wire x1="88.9" y1="17.78" x2="73.66" y2="17.78" width="0.1524" layer="91"/>
 <label x="73.66" y="17.78" size="1.778" layer="95" rot="R180" xref="yes"/>
+</segment>
+<segment>
+<pinref part="R6" gate="G$1" pin="2"/>
+<pinref part="Q1" gate="G$1" pin="E"/>
+<wire x1="50.8" y1="60.96" x2="50.8" y2="63.5" width="0.1524" layer="91"/>
+<label x="53.34" y="60.96" size="1.778" layer="95" xref="yes"/>
+<wire x1="50.8" y1="60.96" x2="53.34" y2="60.96" width="0.1524" layer="91"/>
+<junction x="50.8" y="60.96"/>
 </segment>
 </net>
@@
 <pinref part="GND1" gate="1" pin="GND"/>
 </segment>
+<segment>
+<pinref part="GND3" gate="1" pin="GND"/>
+<pinref part="R6" gate="G$1" pin="1"/>
+<wire x1="50.8" y1="45.72" x2="50.8" y2="50.8" width="0.1524" layer="91"/>
+</segment>
 </net>
 <net name="+12V" class="0">
@@
 <wire x1="38.1" y1="33.02" x2="38.1" y2="38.1" width="0.1524" layer="91"/>
 <pinref part="P+3" gate="1" pin="+12V"/>
-</segment>
-<segment>
-<pinref part="Q1" gate="G$1" pin="C"/>
-<wire x1="50.8" y1="73.66" x2="50.8" y2="78.74" width="0.1524" layer="91"/>
-<pinref part="P+6" gate="1" pin="+12V"/>
 </segment>
 <segment>
@@
 <wire x1="12.7" y1="50.8" x2="15.24" y2="50.8" width="0.1524" layer="91"/>
 <wire x1="12.7" y1="50.8" x2="2.54" y2="50.8" width="0.1524" layer="91"/>
+</segment>
+<segment>
+<pinref part="R5" gate="G$1" pin="2"/>
+<pinref part="P+6" gate="1" pin="+12V"/>
+<wire x1="50.8" y1="88.9" x2="50.8" y2="91.44" width="0.1524" layer="91"/>
 </segment>
 </net>
@@
 </segment>
 </net>
+<net name="N$4" class="0">
+<segment>
+<pinref part="Q1" gate="G$1" pin="C"/>
+<pinref part="R5" gate="G$1" pin="1"/>
+<wire x1="50.8" y1="73.66" x2="50.8" y2="78.74" width="0.1524" layer="91"/>
+</segment>
+</net>

Commit message: Add reset pullup to VDD
Parts:
- added R7: 2k, adafruit:R-US_R0805
Connections:
- net RST: now also R7.1
- net VDD: now also R7.2
Changed lines of the file:
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@@
 <part name="GND3" library="supply1" deviceset="GND" device=""/>
 <part name="R6" library="adafruit" deviceset="R-US_" device="R0805" value="2k"/>
+<part name="VDD3" library="supply1" deviceset="VDD" device=""/>
+<part name="R7" library="adafruit" deviceset="R-US_" device="R0805" value="2k"/>
 </parts>
 <sheets>
@@
 <instance part="GND3" gate="1" x="50.8" y="43.18"/>
 <instance part="R6" gate="G$1" x="50.8" y="55.88" rot="R90"/>
+<instance part="VDD3" gate="G$1" x="60.96" y="81.28"/>
+<instance part="R7" gate="G$1" x="60.96" y="71.12" rot="R90"/>
 </instances>
 <busses>
@@
 <wire x1="50.8" y1="60.96" x2="53.34" y2="60.96" width="0.1524" layer="91"/>
 <junction x="50.8" y="60.96"/>
+<pinref part="R7" gate="G$1" pin="1"/>
+<wire x1="60.96" y1="66.04" x2="53.34" y2="66.04" width="0.1524" layer="91"/>
+<wire x1="53.34" y1="66.04" x2="53.34" y2="60.96" width="0.1524" layer="91"/>
 </segment>
 </net>
@@
 <pinref part="VDD2" gate="G$1" pin="VDD"/>
 </segment>
+<segment>
+<pinref part="R7" gate="G$1" pin="2"/>
+<pinref part="VDD3" gate="G$1" pin="VDD"/>
+<wire x1="60.96" y1="76.2" x2="60.96" y2="78.74" width="0.1524" layer="91"/>
+</segment>
 </net>

Commit message: Tune up boards for printing
Other:
- moved on the sheet: R4
Changed lines of the file:
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@@
 <instance part="P+7" gate="1" x="93.98" y="76.2"/>
 <instance part="VDD2" gate="G$1" x="83.82" y="83.82"/>
-<instance part="R4" gate="G$1" x="7.62" y="50.8"/>
+<instance part="R4" gate="G$1" x="7.62" y="55.88"/>
 <instance part="R5" gate="G$1" x="50.8" y="83.82" rot="R90"/>
 <instance part="GND3" gate="1" x="50.8" y="43.18"/>
@@
 <segment>
 <pinref part="R4" gate="G$1" pin="1"/>
-<wire x1="0" y1="50.8" x2="2.54" y2="50.8" width="0.1524" layer="91"/>
+<wire x1="0" y1="50.8" x2="2.54" y2="55.88" width="0.1524" layer="91"/>
 <pinref part="R4" gate="G$1" pin="2"/>
-<wire x1="12.7" y1="50.8" x2="15.24" y2="50.8" width="0.1524" layer="91"/>
-<wire x1="12.7" y1="50.8" x2="2.54" y2="50.8" width="0.1524" layer="91"/>
+<wire x1="12.7" y1="55.88" x2="15.24" y2="50.8" width="0.1524" layer="91"/>
+<wire x1="12.7" y1="55.88" x2="2.54" y2="55.88" width="0.1524" layer="91"/>
 </segment>
 <segment>
